Commit message: combi 2 scanners + URDF

File: laser_scanners/urdf/att.urdf (robot description, URDF)
Before this commit: robot ATT, 9 links, 8 joints
Joints:
- joint att_to_scanner_left: origin xyz=1.221 -2.880 -0.407 rpy=3.1415923565 0 -0.785398163 -> xyz=1.221 -2.880 -0.407 rpy= 0 3.1415926535 2.35619448
- joint att_to_scanner_right: origin xyz=-1.221 2.880 -0.407 rpy=3.1415923565 0 2.35619449 -> xyz=-1.221 -2.880 -0.407 rpy=0 3.1415923565 0.785398163
